File: atf22v10/atf22v10.kicad_sch (KiCad schematic)
At the start: 25 parts, among them J1 Conn_02x13_Odd_Even, J2 Conn_01x01, J3 Conn_01x01, Q1 2N7000, Q2 2N7000, Q3 BC327, U1 74HCT244, U2 LM7805_TO220, U3 ATF22LV10CQZ

Commit message: Schematic cleanup
Parts:
- J1: value Conn_02x13_Odd_Even -> RPi_GPIO_Header
- J2, J3: footprint SK_Connector:Connector_Banana_THT -> Connector_SK:Connector_Banana_THT
Connections:
- net GPIO14 EDIT renamed GPIO14
- net GPIO15 P/~{V} renamed GPIO15
- net GPIO18 FUSE renamed GPIO18
- net GPIO23 ERASE renamed GPIO23
- net GPIO24 CLOCK renamed GPIO24
- net GPIO25 DIN renamed GPIO25
- net GPIO7 DOUT renamed GPIO7
- net GPIO8 STROBE renamed GPIO8
Other:
- title: (none) -> ATF22V10 Programmer
- moved on the sheet: Q2, R6
Changed lines of the file:
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@@
 (kicad_sch (version 20230121) (generator eeschema)
   (paper "A4")
+  (title_block
+    (title "ATF22V10 Programmer")
+    (date "2024-02-26")
+    (rev "1")
+  )
   (junction (at 187.96 99.06) (diameter 0) (color 0 0 0 0)
   )
@@
     (stroke (width 0) (type default))
   )
-  (wire (pts (xy 154.94 88.9) (xy 154.94 91.44))
+  (wire (pts (xy 154.94 86.36) (xy 154.94 91.44))
     (stroke (width 0) (type default))
   )
@@
     (stroke (width 0) (type default))
   )
-  (wire (pts (xy 165.1 63.5) (xy 165.1 73.66))
+  (wire (pts (xy 165.1 63.5) (xy 165.1 71.12))
     (stroke (width 0) (type default))
   )
@@
     (stroke (width 0) (type default))
   )
-  (wire (pts (xy 154.94 78.74) (xy 157.48 78.74))
+  (wire (pts (xy 154.94 76.2) (xy 157.48 76.2))
     (stroke (width 0) (type default))
   )
@@
     (stroke (width 0) (type default))
   )
-  (wire (pts (xy 139.7 35.56) (xy 139.7 38.1))
-    (stroke (width 0) (type default))
-  )
   (wire (pts (xy 165.1 50.8) (xy 165.1 53.34))
     (stroke (width 0) (type default))
@@
     (stroke (width 0) (type default))
   )
-  (wire (pts (xy 154.94 78.74) (xy 154.94 81.28))
+  (wire (pts (xy 154.94 76.2) (xy 154.94 78.74))
     (stroke (width 0) (type default))
   )
@@
     (stroke (width 0) (type default))
   )
-  (wire (pts (xy 165.1 83.82) (xy 165.1 86.36))
+  (wire (pts (xy 165.1 81.28) (xy 165.1 83.82))
     (stroke (width 0) (type default))
   )
@@
     (stroke (width 0) (type default))
   )
-  (label "GPIO15 P{slash}~{V}" (at 91.44 91.44 0) (fields_autoplaced)
+  (label "GPIO15" (at 91.44 91.44 0) (fields_autoplaced)
     (effects (font (size 1.27 1.27)) (justify left bottom))
   )
-  (label "GPIO23 ERASE" (at 91.44 99.06 0) (fields_autoplaced)
+  (label "GPIO23" (at 91.44 99.06 0) (fields_autoplaced)
     (effects (font (size 1.27 1.27)) (justify left bottom))
   )
@@
     (effects (font (size 1.27 1.27)) (justify left bottom))
   )
-  (label "GPIO7 DOUT" (at 91.44 111.76 0) (fields_autoplaced)
+  (label "GPIO7" (at 91.44 111.76 0) (fields_autoplaced)
     (effects (font (size 1.27 1.27)) (justify left bottom))
   )
-  (label "GPIO14 EDIT" (at 91.44 88.9 0) (fields_autoplaced)
+  (label "GPIO14" (at 91.44 88.9 0) (fields_autoplaced)
     (effects (font (size 1.27 1.27)) (justify left bottom))
   )
-  (label "GPIO24 CLOCK" (at 91.44 101.6 0) (fields_autoplaced)
+  (label "+12V" (at 129.54 38.1 0) (fields_autoplaced)
     (effects (font (size 1.27 1.27)) (justify left bottom))
   )
-  (label "GPIO18 FUSE" (at 91.44 93.98 0) (fields_autoplaced)
+  (label "GPIO24" (at 91.44 101.6 0) (fields_autoplaced)
     (effects (font (size 1.27 1.27)) (justify left bottom))
   )
-  (label "GPIO25 DIN" (at 91.44 106.68 0) (fields_autoplaced)
+  (label "GPIO18" (at 91.44 93.98 0) (fields_autoplaced)
     (effects (font (size 1.27 1.27)) (justify left bottom))
   )
-  (label "GPIO8 STROBE" (at 91.44 109.22 0) (fields_autoplaced)
+  (label "GPIO25" (at 91.44 106.68 0) (fields_autoplaced)
+    (effects (font (size 1.27 1.27)) (justify left bottom))
+  )
+  (label "GPIO8" (at 91.44 109.22 0) (fields_autoplaced)
     (effects (font (size 1.27 1.27)) (justify left bottom))
   )
@@
     )
   )
-  (symbol (lib_id "power:+12V") (at 139.7 35.56 0) (unit 1)
-    (in_bom yes) (on_board yes) (dnp no) (fields_autoplaced)
-    (property "Reference" "#PWR04" (at 139.7 39.37 0)
-      (effects (font (size 1.27 1.27)) hide)
-    )
-    (property "Value" "+12V" (at 139.7 30.48 0)
-      (effects (font (size 1.27 1.27)))
-    )
-    (property "Footprint" "" (at 139.7 35.56 0)
-      (effects (font (size 1.27 1.27)) hide)
-    )
-    (property "Datasheet" "" (at 139.7 35.56 0)
-      (effects (font (size 1.27 1.27)) hide)
-    )
-    (pin "1")
-    (instances
-      (project "atf22v10"
-        (path "/af4d6c20-d19f-4da5-8896-3746f58aa177"
-          (reference "#PWR04") (unit 1)
-        )
-      )
-    )
-  )
   (symbol (lib_id "Device:R") (at 101.6 118.11 180) (unit 1)
     (in_bom yes) (on_board yes) (dnp no)
@@
     )
   )
-  (symbol (lib_id "power:GND") (at 165.1 86.36 0) (mirror y) (unit 1)
-    (in_bom yes) (on_board yes) (dnp no)
-    (property "Reference" "#PWR06" (at 165.1 92.71 0)
-      (effects (font (size 1.27 1.27)) hide)
-    )
-    (property "Value" "GND" (at 165.1 91.44 0)
-      (effects (font (size 1.27 1.27)))
-    )
-    (property "Footprint" "" (at 165.1 86.36 0)
-      (effects (font (size 1.27 1.27)) hide)
-    )
-    (property "Datasheet" "" (at 165.1 86.36 0)
+  (symbol (lib_id "power:GND") (at 165.1 83.82 0) (mirror y) (unit 1)
+    (in_bom yes) (on_board yes) (dnp no)
+    (property "Reference" "#PWR06" (at 165.1 90.17 0)
+      (effects (font (size 1.27 1.27)) hide)
+    )
+    (property "Value" "GND" (at 165.1 88.9 0)
+      (effects (font (size 1.27 1.27)))
+    )
+    (property "Footprint" "" (at 165.1 83.82 0)
+      (effects (font (size 1.27 1.27)) hide)
+    )
+    (property "Datasheet" "" (at 165.1 83.82 0)
       (effects (font (size 1.27 1.27)) hide)
     )
@@
       (effects (font (size 1.27 1.27)))
     )
-    (property "Footprint" "SK_Connector:Connector_Banana_THT" (at 121.92 38.1 0)
+    (property "Footprint" "Connector_SK:Connector_Banana_THT" (at 121.92 38.1 0)
       (effects (font (size 1.27 1.27)) hide)
     )
@@
     )
   )
-  (symbol (lib_id "Transistor_FET:2N7000") (at 162.56 78.74 0) (unit 1)
-    (in_bom yes) (on_board yes) (dnp no)
-    (property "Reference" "Q2" (at 167.64 77.47 0)
+  (symbol (lib_id "Transistor_FET:2N7000") (at 162.56 76.2 0) (unit 1)
+    (in_bom yes) (on_board yes) (dnp no)
+    (property "Reference" "Q2" (at 167.64 74.93 0)
       (effects (font (size 1.27 1.27)) (justify left))
     )
-    (property "Value" "2N7000" (at 167.64 80.01 0)
+    (property "Value" "2N7000" (at 167.64 77.47 0)
       (effects (font (size 1.27 1.27)) (justify left))
     )
-    (property "Footprint" "Package_TO_SOT_THT:TO-92_Inline_Wide" (at 167.64 80.645 0)
+    (property "Footprint" "Package_TO_SOT_THT:TO-92_Inline_Wide" (at 167.64 78.105 0)
       (effects (font (size 1.27 1.27) italic) (justify left) hide)
     )
-    (property "Datasheet" "https://www.vishay.com/docs/70226/70226.pdf" (at 167.64 82.55 0)
+    (property "Datasheet" "https://www.vishay.com/docs/70226/70226.pdf" (at 167.64 80.01 0)
       (effects (font (size 1.27 1.27)) (justify left) hide)
     )
-    (property "Field4" "" (at 162.56 78.74 0)
+    (property "Field4" "" (at 162.56 76.2 0)
       (effects (font (size 1.27 1.27)) hide)
     )
@@
       (effects (font (size 1.27 1.27)))
     )
-    (property "Footprint" "SK_Connector:Connector_Banana_THT" (at 121.92 50.8 0)
+    (property "Footprint" "Connector_SK:Connector_Banana_THT" (at 121.92 50.8 0)
       (effects (font (size 1.27 1.27)) hide)
     )
@@
       (effects (font (size 1.27 1.27)) (justify left))
     )
-    (property "Value" "ATF22LV10CQZ" (at 186.69 110.49 0)
+    (property "Value" "ATF22LV10CQZ" (at 204.47 74.93 0)
       (effects (font (size 1.27 1.27)) (justify left))
     )
@@
     )
   )
-  (symbol (lib_id "Device:R") (at 154.94 85.09 0) (unit 1)
-    (in_bom yes) (on_board yes) (dnp no)
-    (property "Reference" "R6" (at 152.4 83.82 0)
-      (effects (font (size 1.27 1.27)) (justify right))
-    )
-    (property "Value" "47" (at 152.4 86.36 0)
-      (effects (font (size 1.27 1.27)) (justify right))
-    )
-    (property "Footprint" "Resistor_THT:R_Axial_DIN0207_L6.3mm_D2.5mm_P7.62mm_Horizontal" (at 153.162 85.09 90)
-      (effects (font (size 1.27 1.27)) hide)
-    )
-    (property "Datasheet" "~" (at 154.94 85.09 0)
+  (symbol (lib_id "Device:R") (at 154.94 82.55 0) (unit 1)
+    (in_bom yes) (on_board yes) (dnp no)
+    (property "Reference" "R6" (at 152.4 81.28 0)
+      (effects (font (size 1.27 1.27)) (justify right))
+    )
+    (property "Value" "47" (at 152.4 83.82 0)
+      (effects (font (size 1.27 1.27)) (justify right))
+    )
+    (property "Footprint" "Resistor_THT:R_Axial_DIN0207_L6.3mm_D2.5mm_P7.62mm_Horizontal" (at 153.162 82.55 90)
+      (effects (font (size 1.27 1.27)) hide)
+    )
+    (property "Datasheet" "~" (at 154.94 82.55 0)
       (effects (font (size 1.27 1.27)) hide)
     )
@@
   )
   (symbol (lib_id "Connector_Generic:Conn_02x13_Odd_Even") (at 73.66 96.52 0) (unit 1)
-    (in_bom yes) (on_board yes) (dnp no) (fields_autoplaced)
+    (in_bom yes) (on_board yes) (dnp no)
     (property "Reference" "J1" (at 74.93 74.93 0)
       (effects (font (size 1.27 1.27)))
     )
-    (property "Value" "Conn_02x13_Odd_Even" (at 74.93 77.47 0)
-      (effects (font (size 1.27 1.27)))
-    )
+    (property "Value" "RPi_GPIO_Header" (at 74.93 77.47 0)
+      (effects (font (size 1.27 1.27)))
+    )
